File: Sequencer.kicad_pcb (KiCad board)
At the start: 2 copper layers, 80 x 38 mm, 28 parts, among them J1 Screw_Terminal_01x05, J2 Conn_01x02_Female, J3 Conn_01x02_Female, Q1 MMBT3904, Q2 SiHFR320, Q3 MMBF170, Q4 MMBF170, Q5 IRF9540N

Commit message: Heatsink traces
Update
Parts:
- D2: footprint Package_TO_SOT_SMD:SOT-23 -> Diode_SMD:D_SOT-23_ANK
- moved C4 2.68 mm to (119.5, 86.1)
- moved D3 2.10 mm to (116.0, 87.8), turned to 270 degrees
- moved D2 0.13 mm to (111.9, 88.9)
Routing:
- net Net-(D2-Pad1): track 13.1 -> 11.1 mm, vias 2 -> 0
- net Net-(C4-Pad1): track 14.4 -> 13.2 mm
- net Net-(D4-Pad1): track 99.5 -> 100.4 mm, vias 2 -> 4
- net Net-(D2-Pad2): track 3.08 -> 3.81 mm
Other:
- board text added: "A"
- board text added: "V2 9/19"
- board text removed: "V1 8/19"
