File: Sequencer.sch (KiCad schematic (older format))
At the start: 28 parts, among them J1 Screw_Terminal_01x05, J2 Conn_01x02_Female, J3 Conn_01x02_Female, Q1 MMBT3904, Q2 SiHFR320, Q3 MMBF170, Q4 MMBF170, Q5 IRF9540N

Commit message: Heatsink traces
Update
Parts:
- D2: footprint Package_TO_SOT_SMD:SOT-23 -> Diode_SMD:D_SOT-23_ANK
- R4: value 1k -> 4.7k
Changed lines of the file:
@@
 F 0 "D2" H 5250 3284 50  0000 C CNN
 F 1 "BZX84C5V1LT1G" H 5250 3375 50  0000 C CNN
-F 2 "Package_TO_SOT_SMD:SOT-23" H 5250 3500 50  0001 C CNN
+F 2 "Diode_SMD:D_SOT-23_ANK" H 5250 3500 50  0001 C CNN
 F 3 "~" H 5250 3500 50  0001 C CNN
 	1    5250 3500
@@
 U 1 1 5D5BABF8
 P 6350 4400
-F 0 "R5" H 6200 4300 50  0000 C CNN
-F 1 "10k" H 6200 4400 50  0000 C CNN
+F 0 "R5" H 6200 4400 50  0000 C CNN
+F 1 "10k" H 6200 4500 50  0000 C CNN
 F 2 "Resistor_SMD:R_0805_2012Metric" V 6280 4400 50  0001 C CNN
 F 3 "~" H 6350 4400 50  0001 C CNN
@@
 Wire Wire Line
 	6600 3850 6650 3850
-Connection ~ 6650 3850
 $Comp
 L Device:R R4
 U 1 1 5D5C0472
 P 5650 4250
-F 0 "R4" V 5500 4150 50  0000 C CNN
-F 1 "1k" V 5550 4250 50  0000 C CNN
+F 0 "R4" V 5750 4250 50  0000 C CNN
+F 1 "4.7k" V 5550 4250 50  0000 C CNN
 F 2 "Resistor_SMD:R_0805_2012Metric" V 5580 4250 50  0001 C CNN
 F 3 "~" H 5650 4250 50  0001 C CNN
@@
 U 1 1 5D5C6CA8
 P 6100 4250
-F 0 "D4" H 6200 4350 50  0000 C CNN
+F 0 "D4" H 6250 4200 50  0000 C CNN
 F 1 "LED" H 6100 4400 50  0000 C CNN
 F 2 "LED_SMD:LED_0805_2012Metric_Castellated" H 6100 4250 50  0001 C CNN
@@
 	6800 3750 7250 3750
 Wire Wire Line
-	6650 3850 7250 3850
-Wire Wire Line
 	6500 3950 7250 3950
 Wire Wire Line
@@
 	1    0    0    -1
 $EndComp
+Connection ~ 6650 3850
+Wire Wire Line
+	6650 3850 7250 3850
 $EndSCHEMATC
